File: NMPavi280wires.sch (EAGLE design)
At the start: 5 parts, among them J1 22-27-2061-06, J2 22-27-2081-08, J3 22-27-2021-02

Commit message: Add files via upload
Parts:
- renumbered J1 to SDCARD, J2 to BMP388, J3 to BATTERY, X1 to BMP280
